File: Pcb/Pcb.sch (KiCad schematic (older format))
At the start: 133 parts, among them J1 TRRS, Q1 2N7002, SW1 SW_Push, SW10 SW_Push, SW11 SW_Push, SW12 SW_Push, SW13 SW_Push, SW14 SW_Push, SW15 SW_Push, SW16 SW_Push, SW17 SW_Push, SW18 SW_Push, SW19 SW_Push, SW2 SW2, SW20 SW_Push, SW21 SW_Push, SW22 SW_Push, SW23 SW_Push, SW24 SW_Push, SW25 SW_Push, SW26 SW_Push, SW27 SW_Push, SW28 SW_Push, SW29 SW_Push, SW3 SW_Push, SW4 SW_Push, SW5 SW_Push, SW6 SW_Push, SW7 SW_Push, SW8 SW_Push, SW9 SW_Push, U1 ProMicro

Commit message: Add footprints for resistors and jumpers
Parts:
- JP1, JP2, JP3, JP4: footprint (none) -> Used_Footprints:Jumper_SMD
- R29, R30: footprint (none) -> Used_Footprints:Resistor_Hybrid_1205
Changed lines of the file:
@@
 F 0 "R29" H 855 1290 50  0000 L CNN
 F 1 "4.7K" H 855 1200 50  0000 L CNN
-F 2 "" H 810 1245 50  0001 C CNN
+F 2 "Used_Footprints:Resistor_Hybrid_1205" H 810 1245 50  0001 C CNN
 F 3 "~" H 810 1245 50  0001 C CNN
 	1    810  1245
@@
 F 0 "R30" H 855 1590 50  0000 L CNN
 F 1 "4.7K" H 855 1500 50  0000 L CNN
-F 2 "" H 810 1545 50  0001 C CNN
+F 2 "Used_Footprints:Resistor_Hybrid_1205" H 810 1545 50  0001 C CNN
 F 3 "~" H 810 1545 50  0001 C CNN
 	1    810  1545
@@
 	810  1445 1240 1445
 $Comp
-L power:VCC #PWR?
+L power:VCC #PWR0101
 U 1 1 5E5BBB5F
 P 810 1105
-F 0 "#PWR?" H 810 955 50  0001 C CNN
+F 0 "#PWR0101" H 810 955 50  0001 C CNN
 F 1 "VCC" H 810 1250 50  0000 C CNN
 F 2 "" H 810 1105 50  0001 C CNN
@@
 $EndComp
 $Comp
-L power:VCC #PWR?
+L power:VCC #PWR0102
 U 1 1 5E5BC852
 P 810 1685
-F 0 "#PWR?" H 810 1535 50  0001 C CNN
+F 0 "#PWR0102" H 810 1535 50  0001 C CNN
 F 1 "VCC" H 810 1835 50  0000 C CNN
 F 2 "" H 810 1685 50  0001 C CNN
@@
 F 0 "JP1" H 1520 2490 50  0000 C CNN
 F 1 "Jumper" H 1525 2605 50  0000 C CNN
-F 2 "" H 1525 2525 50  0001 C CNN
+F 2 "Used_Footprints:Jumper_SMD" H 1525 2525 50  0001 C CNN
 F 3 "~" H 1525 2525 50  0001 C CNN
 	1    1525 2525
@@
 F 0 "JP2" H 1520 2690 50  0000 C CNN
 F 1 "Jumper" H 1525 2805 50  0000 C CNN
-F 2 "" H 1525 2725 50  0001 C CNN
+F 2 "Used_Footprints:Jumper_SMD" H 1525 2725 50  0001 C CNN
 F 3 "~" H 1525 2725 50  0001 C CNN
 	1    1525 2725
@@
 F 0 "JP3" H 1520 2890 50  0000 C CNN
 F 1 "Jumper" H 1525 3005 50  0000 C CNN
-F 2 "" H 1525 2925 50  0001 C CNN
+F 2 "Used_Footprints:Jumper_SMD" H 1525 2925 50  0001 C CNN
 F 3 "~" H 1525 2925 50  0001 C CNN
 	1    1525 2925
@@
 F 0 "JP4" H 1520 3090 50  0000 C CNN
 F 1 "Jumper" H 1525 3205 50  0000 C CNN
-F 2 "" H 1525 3125 50  0001 C CNN
+F 2 "Used_Footprints:Jumper_SMD" H 1525 3125 50  0001 C CNN
 F 3 "~" H 1525 3125 50  0001 C CNN
 	1    1525 3125
@@
 	1775 3125 1725 3125
 $Comp
-L power:GND #PWR?
+L power:GND #PWR0103
 U 1 1 5E653D30
 P 880 3070
-F 0 "#PWR?" H 880 2820 50  0001 C CNN
+F 0 "#PWR0103" H 880 2820 50  0001 C CNN
 F 1 "GND" V 880 2950 50  0000 R CNN
 F 2 "" H 880 3070 50  0001 C CNN
@@
 	1155 3070 1155 2975
 $Comp
-L power:VCC #PWR?
+L power:VCC #PWR0104
 U 1 1 5E65ED2C
 P 880 3220
-F 0 "#PWR?" H 880 3070 50  0001 C CNN
+F 0 "#PWR0104" H 880 3070 50  0001 C CNN
 F 1 "VCC" V 875 3345 50  0000 L CNN
 F 2 "" H 880 3220 50  0001 C CNN
