File: jiran-hotswap/pcb.kicad_pcb (KiCad board)
At the start: 2 copper layers, 152.3 x 104.7 mm, 103 parts, among them J1 TRRS, SW1 SW_Push, SW10 SW_Push, SW11 SW_Push, SW12 SW_Push, SW13 SW_Push, SW14 SW_Push, SW15 SW_Push, SW16 SW_Push, SW17 SW_Push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

Commit message: add new logo silkscreen
Parts:
- added LG1: Silk_Logo_New, Used_Footprints:Silk_Logo_New, F.Cu at (206.2, 83.9)
- added LG2: Silk_Logo_New, Used_Footprints:Silk_Logo_New, B.Cu at (206.1, 83.9)
