File: jiran-hotswap/pcb.sch (KiCad schematic (older format))
At the start: 103 parts, among them J1 TRRS, SW1 SW_Push, SW10 SW_Push, SW11 SW_Push, SW12 SW_Push, SW13 SW_Push, SW14 SW_Push, SW15 SW_Push, SW16 SW_Push, SW17 SW_Push, SW18 SW_Push, SW19 SW_Push, SW2 SW2, SW20 SW_Push, SW21 SW_Push, SW22 SW_Push, SW23 SW_Push, SW24 SW_Push, SW25 SW_Push, SW26 SW_Push, SW27 SW_Push, SW28 SW_Push, SW29 SW_Push, SW3 SW_Push, SW4 SW_Push, SW5 SW_Push, SW6 SW_Push, SW7 SW_Push, SW8 SW_Push, SW9 SW_Push, U1 ProMicro

Commit message: Route tracks
Parts:
- D1, D10, D11, D12, D13, D14, D15, D16, D17, D18, D19, D2, D20, D21, D22, D23, D24, D25, D26, D27, D28, D3, D4, D5, D6, D7, D8, D9: footprint Used_Footprints:Diode_Hybrid_SOD-123 -> Used_Footprints:Diode_SMD_SOD-123
- L1, L10, L11, L12, L13, L14, L15, L16, L17, L18, L19, L2, L20, L21, L22, L23, L24, L25, L26, L27, L28, L3, L4, L5, L6, L7, L8, L9: footprint (none) -> Used_Footprints:SK6812MINI
- SW1, SW10, SW11, SW12, SW13, SW14, SW15, SW16, SW17, SW18, SW19, SW2, SW20, SW21, SW22, SW23, SW24, SW25, SW26, SW27, SW28, SW3, SW4, SW5, SW6, SW7, SW8, SW9: footprint Used_Footprints:Switch_MxAlpsChoc_MillMax_1u -> Used_Footprints:Switch_Mx_Hotswap_1u
Connections:
- net labels removed: LED

Commit message: Remove RGB leds
Parts:
- removed L1, L10, L11, L12, L13, L14, L15, L16, L17, L18, L19, L2, L20, L21, L22, L23, L24, L25, L26, L27, L28, L3, L4, L5, L6, L7, L8, L9: SK6812MINI-kbd, Used_Footprints:SK6812MINI, symbol corne-classic-rescue:SK6812MINI-kbd
Connections:
- net labels removed: RGB
- wire segments 269 -> 82
