File: jiran-hotswap/jiran-hotswap.sch (KiCad schematic (older format))
At the start: 132 parts, among them J1 TRRS, Q1 2N7002, SW1 SW_Push, SW10 SW_Push, SW11 SW_Push, SW12 SW_Push, SW13 SW_Push, SW14 SW_Push, SW15 SW_Push, SW16 SW_Push, SW17 SW_Push, SW18 SW_Push, SW19 SW_Push, SW2 SW_Push, SW20 SW_Push, SW21 SW_Push, SW22 SW_Push, SW23 SW_Push, SW24 SW_Push, SW25 SW_Push, SW26 SW_Push, SW27 SW_Push, SW28 SW_Push, SW29 SW_Push, SW3 SW_Push, SW4 SW_Push, SW5 SW_Push, SW6 SW_Push, SW7 SW_Push, SW8 SW_Push, SW9 SW_Push, U1 ProMicro

Commit message: Remove LED block
Parts:
- removed D29, D30, D31, D32, D33, D34, D35, D36, D37, D38, D39, D40, D41, D42, D43, D44, D45, D46, D47, D48, D49, D50, D51, D52, D53, D54, D55, D56: LED_Small, used_footprints:LED_THT, symbol Device:LED_Small
- removed G1, G2: LOGO, used_footprints:Silk_Logotype, symbol jiran-classic-rescue:LOGO-jiran
- removed Q1: 2N7002, used_footprints:Mosfet_SMD_Dual_SOT-23, symbol Transistor_FET:2N7002
- removed R1, R10, R11, R12, R13, R14, R15, R16, R17, R18, R19, R2, R20, R21, R22, R23, R24, R25, R26, R27, R28, R3, R4, R5, R6, R7, R8, R9: 300R, used_footprints:Resistor_Hybrid_1205, symbol Device:R_Small
- removed R31: 100k, used_footprints:Resistor_Hybrid_1205, symbol Device:R_Small
- added G1, G2: logo-jiran-hotswap, used_footprints:Silk_Logo_Hotswap, symbol jiran:logo-jiran-hotswap
- J1: symbol jiran-classic-rescue:MJ-4PP-9-kbd-Pcb-rescue -> jiran-hotswap-rescue:MJ-4PP-9-kbd-Pcb-rescue-jiran-classic-rescue-jiran-hotswap-rescue
- SW1, SW10, SW11, SW12, SW13, SW14, SW15, SW16, SW17, SW18, SW19, SW2, SW20, SW21, SW22, SW23, SW24, SW25, SW26, SW27, SW28, SW3, SW4, SW5, SW6, SW7, SW8, SW9: footprint used_footprints:Switch_MxAlpsChoc_MillMax_1u -> used_footprints:Switch_Mx_Hotswap_1u
- U1: symbol jiran-classic-rescue:ProMicro-kbd-Pcb-rescue -> jiran-hotswap-rescue:ProMicro-kbd-Pcb-rescue-jiran-classic-rescue-jiran-hotswap-rescue
Other:
- moved on the sheet: HC1, HC2, HM1, HM2, HM3, HM4, HM5
