File: jiran-classic/Pcb.kicad_pcb (KiCad board)
At the start: 2 copper layers, 152.3 x 104.7 mm, 135 parts, among them J1 TRRS, Q1 2N7002, SW1 SW_Push, SW10 SW_Push, SW11 SW_Push, SW12 SW_Push, SW13 SW_Push, SW14 SW_Push, SW15 SW_Push, SW16 SW_Push, SW17 SW_Push, SW18 SW_Push, SW19 SW_Push, SW2 SW2, SW20 SW_Push, SW21 SW_Push, SW22 SW_Push, SW23 SW_Push, SW24 SW_Push, SW25 SW_Push, SW26 SW_Push, SW27 SW_Push, SW28 SW_Push, SW29 SW_Push, SW3 SW_Push, SW4 SW_Push, SW5 SW_Push, SW6 SW_Push, SW7 SW_Push, SW8 SW_Push, SW9 SW_Push, U1 ProMicro

Commit message: Remove breakoff future
Parts:
- removed the HM4 at (153.3, 51.5)
- removed the HM5 at (153.3, 70.6)
- moved HM3 38.3 mm to (153.3, 51.5)
- moved HM2 19.0 mm to (191.4, 55.0)
- renumbered HM6 to HM4, HM7 to HM5, HM8 to HM6
Routing:
- net VCC: track 629.7 -> 0.00 mm, vias 1 -> 0
- net /LEDOut: track 587.6 -> 0.00 mm
- net /rowE: track 262.4 -> 0.00 mm, vias 1 -> 0
- net /col0: track 231.9 -> 0.00 mm
- net /col1: track 199.0 -> 0.00 mm, vias 1 -> 0
- net /rowA: track 197.9 -> 0.00 mm, vias 3 -> 0
- net /col3: track 196.4 -> 0.00 mm, vias 2 -> 0
- net /rowD: track 191.5 -> 0.00 mm
- net /col4: track 176.9 -> 0.00 mm
- net /rowB: track 176.6 -> 0.00 mm, vias 1 -> 0
- net /col2: track 162.4 -> 0.00 mm
- net /rowC: track 156.7 -> 0.00 mm, vias 1 -> 0
- net /col5: track 134.3 -> 0.00 mm
- net GND: track 80.5 -> 0.00 mm, vias 1 -> 0
- net SDA: track 65.0 -> 0.00 mm, vias 1 -> 0
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Other:
- outline, holes or cut-outs redrawn

Commit message: Add tracks
Parts:
- D1, D10, D11, D12, D13, D14, D15, D16, D17, D18, D19, D2, D20, D21, D22, D23, D24, D25, D26, D27, D28, D3, D4, D5, D6, D7, D8, D9: footprint Used_Footprints:Diode_Hybrid_SOD-123 -> used_footprints:Diode_Hybrid_SOD-123
- D29, D30, D31, D32, D33, D34, D35, D36, D37, D38, D39, D40, D41, D42, D43, D44, D45, D46, D47, D48, D49, D50, D51, D52, D53, D54, D55, D56: footprint Used_Footprints:LED_THT_1.8mm -> used_footprints:LED_THT
- HC1, HC2: footprint Used_Footprints:Hole_Cover_M2 -> used_footprints:Hole_Cover_M2
- HM1, HM2, HM3, HM4, HM5, HM6: footprint Used_Footprints:Hole_Mount_M4 -> used_footprints:Hole_Mount_M4
- J1: footprint Used_Footprints:TRSS_DUAL_THT -> used_footprints:TRSS_DUAL_THT
- JP1, JP2, JP3, JP4: footprint Used_Footprints:Jumper_SMD -> used_footprints:Jumper_SMD
- Q1: footprint Used_Footprints:Mosfet_SMD_Dual_SOT-23 -> used_footprints:Mosfet_SMD_Dual_SOT-23
- R1, R10, R11, R12, R13, R14, R15, R16, R17, R18, R19, R2, R20, R21, R22, R23, R24, R25, R26, R27, R28, R29, R3, R30, R31, R4, R5, R6, R7, R8, R9: footprint Used_Footprints:Resistor_Hybrid_1205 -> used_footprints:Resistor_Hybrid_1205
- SW1, SW10, SW11, SW12, SW13, SW14, SW15, SW16, SW17, SW18, SW19, SW20, SW21, SW22, SW23, SW24, SW25, SW26, SW27, SW28, SW3, SW4, SW5, SW6, SW7, SW8, SW9: footprint Used_Footprints:Switch_MxAlpsChoc_MillMax_1u -> used_footprints:Switch_MxAlpsChoc_MillMax_1u
- SW2: value SW2 -> SW_Push; footprint Used_Footprints:Switch_MxAlpsChoc_MillMax_1u -> used_footprints:Switch_MxAlpsChoc_MillMax_1u
- SW29: footprint Used_Footprints:Switch_Reset_THT -> used_footprints:Switch_Reset_THT
- U1: footprint Used_Footprints:ProMicro_Dual -> used_footprints:ProMicro_Dual
- moved HM4 19.1 mm to (115.2, 62.2)
Routing:
- net VCC: track 0.00 -> 610.0 mm, vias 0 -> 1
- net /LEDOut: track 0.00 -> 579.9 mm
- net /rowE: track 0.00 -> 243.7 mm, vias 0 -> 5
- net /col0: track 0.00 -> 230.2 mm
- net /rowD: track 0.00 -> 201.2 mm, vias 0 -> 1
- net /rowA: track 0.00 -> 188.9 mm, vias 0 -> 1
- net /rowB: track 0.00 -> 181.5 mm, vias 0 -> 1
- net /col1: track 0.00 -> 180.8 mm
- net /col3: track 0.00 -> 173.5 mm
- net /col2: track 0.00 -> 173.0 mm
- net /rowC: track 0.00 -> 155.8 mm, vias 0 -> 1
- net /col4: track 0.00 -> 154.3 mm
- net /col5: track 0.00 -> 141.6 mm
- net GND: track 0.00 -> 85.7 mm, vias 0 -> 1
- net /RST: track 0.00 -> 73.8 mm, vias 0 -> 1
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