File: jiran-classic/Pcb.kicad_pcb (KiCad board)
At the start: 2 copper layers, 152.3 x 104.7 mm, 132 parts, among them J1 TRRS, Q1 2N7002, SW1 SW_Push, SW10 SW_Push, SW11 SW_Push, SW12 SW_Push, SW13 SW_Push, SW14 SW_Push, SW15 SW_Push, SW16 SW_Push, SW17 SW_Push, SW18 SW_Push, SW19 SW_Push, SW2 SW_Push, SW20 SW_Push, SW21 SW_Push, SW22 SW_Push, SW23 SW_Push, SW24 SW_Push, SW25 SW_Push, SW26 SW_Push, SW27 SW_Push, SW28 SW_Push, SW29 SW_Push, SW3 SW_Push, SW4 SW_Push, SW5 SW_Push, SW6 SW_Push, SW7 SW_Push, SW8 SW_Push, SW9 SW_Push, U1 ProMicro

Commit message: Remove all tracks
Routing:
- net VCC: track 610.0 -> 0.00 mm, vias 1 -> 0
- net /LEDOut: track 579.9 -> 0.00 mm
- net /rowE: track 243.7 -> 0.00 mm, vias 5 -> 0
- net /col0: track 230.2 -> 0.00 mm
- net /rowD: track 201.2 -> 0.00 mm, vias 1 -> 0
- net /rowA: track 188.9 -> 0.00 mm, vias 1 -> 0
- net /rowB: track 181.5 -> 0.00 mm, vias 1 -> 0
- net /col1: track 180.8 -> 0.00 mm
- net /col3: track 173.5 -> 0.00 mm
- net /col2: track 173.0 -> 0.00 mm
- net /rowC: track 155.8 -> 0.00 mm, vias 1 -> 0
- net /col4: track 154.3 -> 0.00 mm
- net /col5: track 141.6 -> 0.00 mm
- net GND: track 85.7 -> 0.00 mm, vias 1 -> 0
- net /RST: track 73.8 -> 0.00 mm, vias 1 -> 0
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
Commit message: Fill all zones
Routing:
- net VCC: track 0.00 -> 606.9 mm
- net /LEDOut: track 0.00 -> 579.6 mm
- net /rowE: track 0.00 -> 264.9 mm, vias 0 -> 1
- net /col0: track 0.00 -> 231.6 mm
- net /col3: track 0.00 -> 182.8 mm, vias 0 -> 1
- net /rowA: track 0.00 -> 181.4 mm
- net /col1: track 0.00 -> 180.6 mm
- net /rowD: track 0.00 -> 178.9 mm
- net /col4: track 0.00 -> 169.3 mm
- net /col2: track 0.00 -> 167.0 mm
- net /rowB: track 0.00 -> 165.4 mm, vias 0 -> 1
- net /rowC: track 0.00 -> 157.2 mm, vias 0 -> 1
- net /col5: track 0.00 -> 143.2 mm, vias 0 -> 2
- net GND: track 0.00 -> 103.7 mm
- net SDA: track 0.00 -> 64.7 mm, vias 0 -> 1
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