File: jiran-cherry/jiran-cherry.sch (KiCad schematic (older format))
At the start: 74 parts, among them J1 TRRS, SW1 SW_Push, SW10 SW_Push, SW11 SW_Push, SW12 SW_Push, SW13 SW_Push, SW14 SW_Push, SW15 SW_Push, SW16 SW_Push, SW17 SW_Push, SW18 SW_Push, SW19 SW_Push, SW2 SW_Push, SW20 SW_Push, SW21 SW_Push, SW22 SW_Push, SW23 SW_Push, SW24 SW_Push, SW25 SW_Push, SW26 SW_Push, SW27 SW_Push, SW28 SW_Push, SW29 SW_Push, SW3 SW_Push, SW4 SW_Push, SW5 SW_Push, SW6 SW_Push, SW7 SW_Push, SW8 SW_Push, SW9 SW_Push, U1 ProMicro

Commit message: Update symbol logo
Parts:
- removed G1, G2: logo-jiran-hotswap, used_footprints:Silk_Logo_Hotswap, symbol jiran:logo-jiran-hotswap
- added G1, G2: logo-jiran-cherry, symbol jiran:logo-jiran-cherry
- J1: symbol jiran-hotswap-rescue:MJ-4PP-9-kbd-Pcb-rescue-jiran-classic-rescue-jiran-hotswap-rescue -> jiran-cherry-rescue:MJ-4PP-9-kbd-Pcb-rescue-jiran-classic-rescue-jiran-hotswap-rescue-jiran-hotswap-rescue
- U1: symbol jiran-hotswap-rescue:ProMicro-kbd-Pcb-rescue-jiran-classic-rescue-jiran-hotswap-rescue -> jiran-cherry-rescue:ProMicro-kbd-Pcb-rescue-jiran-classic-rescue-jiran-hotswap-rescue-jiran-hotswap-rescue
Changed lines of the file:
@@
 $EndComp
 $Comp
-L jiran-hotswap-rescue:MJ-4PP-9-kbd-Pcb-rescue-jiran-classic-rescue-jiran-hotswap-rescue J1
+L jiran-cherry-rescue:MJ-4PP-9-kbd-Pcb-rescue-jiran-classic-rescue-jiran-hotswap-rescue-jiran-hotswap-rescue J1
 U 1 1 5DBFACF7
 P 955 2900
@@
 Connection ~ 1240 1145
 $Comp
-L jiran-hotswap-rescue:ProMicro-kbd-Pcb-rescue-jiran-classic-rescue-jiran-hotswap-rescue U1
+L jiran-cherry-rescue:ProMicro-kbd-Pcb-rescue-jiran-classic-rescue-jiran-hotswap-rescue-jiran-hotswap-rescue U1
 U 1 1 5DAA926E
 P 1940 1695
@@
 	2640 1045 2830 1045
 $Comp
-L jiran:logo-jiran-hotswap G1
-U 1 1 5FA214AC
+L jiran:logo-jiran-cherry G1
+U 1 1 5FA1704C
 P 8750 950
 F 0 "G1" H 8700 1200 60  0000 L CNN
-F 1 "logo-jiran-hotswap" H 8750 700 60  0001 C CNN
-F 2 "used_footprints:Silk_Logo_Hotswap" H 8750 950 50  0001 C CNN
+F 1 "logo-jiran-cherry" H 8750 700 60  0001 C CNN
+F 2 "" H 8750 950 50  0001 C CNN
 F 3 "" H 8750 950 50  0001 C CNN
 	1    8750 950
@@
 $EndComp
 $Comp
-L jiran:logo-jiran-hotswap G2
-U 1 1 5FA2276E
+L jiran:logo-jiran-cherry G2
+U 1 1 5FA17C36
 P 9200 950
 F 0 "G2" H 9150 1200 60  0000 L CNN
-F 1 "logo-jiran-hotswap" H 9200 700 60  0001 C CNN
-F 2 "used_footprints:Silk_Logo_Hotswap" H 9200 950 50  0001 C CNN
+F 1 "logo-jiran-cherry" H 9200 700 60  0001 C CNN
+F 2 "" H 9200 950 50  0001 C CNN
 F 3 "" H 9200 950 50  0001 C CNN
 	1    9200 950

Commit message: Assign PCB footprints
Parts:
- G1, G2: footprint (none) -> used_footprints:Silk_Logo_Cherry
Changed lines of the file:
@@
 F 0 "G1" H 8700 1200 60  0000 L CNN
 F 1 "logo-jiran-cherry" H 8750 700 60  0001 C CNN
-F 2 "" H 8750 950 50  0001 C CNN
+F 2 "used_footprints:Silk_Logo_Cherry" H 8750 950 50  0001 C CNN
 F 3 "" H 8750 950 50  0001 C CNN
 	1    8750 950
@@
 F 0 "G2" H 9150 1200 60  0000 L CNN
 F 1 "logo-jiran-cherry" H 9200 700 60  0001 C CNN
-F 2 "" H 9200 950 50  0001 C CNN
+F 2 "used_footprints:Silk_Logo_Cherry" H 9200 950 50  0001 C CNN
 F 3 "" H 9200 950 50  0001 C CNN
 	1    9200 950
