File: jiran-cherry/jiran-cherry.kicad_pcb (KiCad board)
At the start: 2 copper layers, 152.3 x 104.7 mm, 74 parts, among them J1 TRRS, SW1 SW_Push, SW10 SW_Push, SW11 SW_Push, SW12 SW_Push, SW13 SW_Push, SW14 SW_Push, SW15 SW_Push, SW16 SW_Push, SW17 SW_Push, SW18 SW_Push, SW19 SW_Push, SW2 SW_Push, SW20 SW_Push, SW21 SW_Push, SW22 SW_Push, SW23 SW_Push, SW24 SW_Push, SW25 SW_Push, SW26 SW_Push, SW27 SW_Push, SW28 SW_Push, SW29 SW_Push, SW3 SW_Push, SW4 SW_Push, SW5 SW_Push, SW6 SW_Push, SW7 SW_Push, SW8 SW_Push, SW9 SW_Push, U1 ProMicro

Commit message: Route tracks
Routing:
- net /rowE: track 0.00 -> 225.4 mm
- net /col0: track 0.00 -> 223.5 mm
- net /col3: track 0.00 -> 180.8 mm, vias 0 -> 1
- net /col1: track 0.00 -> 180.6 mm
- net /rowA: track 0.00 -> 164.7 mm, vias 0 -> 1
- net /col2: track 0.00 -> 164.7 mm, vias 0 -> 2
- net /col4: track 0.00 -> 159.1 mm, vias 0 -> 1
- net /rowD: track 0.00 -> 158.7 mm
- net /rowB: track 0.00 -> 151.4 mm
- net /col5: track 0.00 -> 141.4 mm, vias 0 -> 1
- net /rowC: track 0.00 -> 140.8 mm
- net GND: track 0.00 -> 72.3 mm
- net SDA: track 0.00 -> 62.3 mm, vias 0 -> 1
- net SCL: track 0.00 -> 60.0 mm, vias 0 -> 2
- net VCC: track 0.00 -> 56.5 mm
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